File: Northstar Protoboard/Northstar Protoboard.kicad_pcb (KiCad board)
At the start: 2 copper layers, 76.3 x 139.9 mm, 809 parts, among them J1 Conn_02x15_Odd_Even, J10 IO A0, J11 I_3, J12 I_1, J13 I_2, J14 enable, J15 O_5, J16 O_3, J17 D3, J18 D2, J19 D4, J2 12v, J20 D5, J21 D6, J22 D1, J23 D0, J24 D7, J25 9v, J26 -9v, J27 direction, J28 IO INT, J29 O_4, J3 5v, J30 O_2, J31 O_1, J32 SELECT, J33 RES, J34 8MHz, J35 IO A1, J36 IO A3, J37 IO A2, J38 ID REQ, J39 13, J4 GND, J40 DB25_Female, J41 25, J42 12, J43 24, J44 11, J45 23, J46 10, J47 22, J48 9, J49 21, J5 -12v, J50 8, J51 20, J52 7, J53 19, J54 6, J55 18, J56 5, J57 17, J58 4, J59 16, J6 I_5, J60 3, J61 15, J62 2, J63 14, J64 1, J65 GND, J66 5v, J7 I_4, J8 BWR, J9 BRD, U1 LM7909_TO220, U2 LM7809_TO220, U3 74LHCT45, U4 74LHCT45, U5 74LHCT45

Commit message: generated gerbers
Routing:
- net GND: track 623.0 -> 621.9 mm
- net +5V: track 490.5 -> 489.8 mm
