File: Northstar SIO - update/Northstar SIO.kicad_pcb (KiCad board)
At the start: 2 copper layers, 76.3 x 139.9 mm, 56 parts, among them J1 DB25_Female, J1A1 CLOCK, J2 Conn_02x15_Odd_Even, J3A1 CONFIG, U1B1 LS161, U1C1 LS161, U1D1 LS161, U1E1 LS174, U2A1 1489, U2B1 LS04, U2C1 LS109, U2D1 LS175, U2E1 LS243, U3B1 LS00, U3C1 LS138, U3D1 LS03, U3E1 LS243, U4A1 1488, U4E1 8251A

Commit message: generated gerbers
Routing:
- net /C: track 75.9 -> 74.2 mm
- net Net-(J3A1-Pad4): track 84.5 -> 85.0 mm
Changed lines of the file:
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@@
       (layerselection 0x00010fc_ffffffff)
       (disableapertmacros false)
-      (usegerberextensions false)
+      (usegerberextensions true)
       (usegerberattributes true)
       (usegerberadvancedattributes true)
@@
       (plotinvisibletext false)
       (sketchpadsonfab false)
-      (subtractmaskfromsilk false)
+      (subtractmaskfromsilk true)
       (outputformat 1)
       (mirror false)
-      (drillshape 1)
+      (drillshape 0)
       (scaleselection 1)
-      (outputdirectory "")
+      (outputdirectory "Northstar SIO-gerbers")
     )
   )
@@
     (fp_line (start -1.37 -1.37) (end 6.37 -1.37) (layer "F.SilkS") (width 0.12))
     (fp_line (start 6.37 -1.37) (end 6.37 1.37) (layer "F.SilkS") (width 0.12))
-    (fp_line (start -1.5 -1.5) (end -1.5 1.5) (layer "F.CrtYd") (width 0.05))
     (fp_line (start -1.5 1.5) (end 6.5 1.5) (layer "F.CrtYd") (width 0.05))
+    (fp_line (start -1.5 -1.5) (end -1.5 1.5) (layer "F.CrtYd") (width 0.05))
     (fp_line (start 6.5 1.5) (end 6.5 -1.5) (layer "F.CrtYd") (width 0.05))
     (fp_line (start 6.5 -1.5) (end -1.5 -1.5) (layer "F.CrtYd") (width 0.05))
@@
   (segment (start 140.462 98.298) (end 145.034 98.298) (width 0.25) (layer "F.Cu") (net 19))
   (segment (start 145.034 98.298) (end 147.828 95.504) (width 0.25) (layer "F.Cu") (net 19))
-  (segment (start 141.732 60.706) (end 140.462 59.436) (width 0.25) (layer "B.Cu") (net 19))
-  (segment (start 142.5575 52.3875) (end 143.51 51.435) (width 0.25) (layer "B.Cu") (net 19))
-  (segment (start 141.00952 53.93548) (end 142.5575 52.3875) (width 0.25) (layer "B.Cu") (net 19))
   (segment (start 144.877307 60.706) (end 141.732 60.706) (width 0.25) (layer "B.Cu") (net 19))
+  (segment (start 147.828 63.656693) (end 144.877307 60.706) (width 0.25) (layer "B.Cu") (net 19))
   (segment (start 146.246 78.08) (end 147.828 76.498) (width 0.25) (layer "B.Cu") (net 19))
-  (segment (start 140.462 54.483) (end 142.5575 52.3875) (width 0.25) (layer "B.Cu") (net 19))
-  (segment (start 140.462 59.436) (end 140.462 54.483) (width 0.25) (layer "B.Cu") (net 19))
+  (segment (start 140.462 53.594) (end 142.621 51.435) (width 0.25) (layer "B.Cu") (net 19))
   (segment (start 147.828 76.498) (end 147.828 63.656693) (width 0.25) (layer "B.Cu") (net 19))
-  (segment (start 147.828 63.656693) (end 144.877307 60.706) (width 0.25) (layer "B.Cu") (net 19))
+  (segment (start 140.462 59.436) (end 140.462 53.594) (width 0.25) (layer "B.Cu") (net 19))
+  (segment (start 142.621 51.435) (end 143.51 51.435) (width 0.25) (layer "B.Cu") (net 19))
+  (segment (start 141.732 60.706) (end 140.462 59.436) (width 0.25) (layer "B.Cu") (net 19))
   (segment (start 141.986 54.61) (end 135.89 54.61) (width 0.25) (layer "F.Cu") (net 23))
   (via (at 135.89 54.61) (size 0.8) (drill 0.4) (layers "F.Cu" "B.Cu") (net 23))
@@
   (segment (start 119.7003 46.355) (end 118.4303 45.085) (width 0.25) (layer "F.Cu") (net 59))
   (segment (start 121.285 55.245) (end 134.230386 55.245) (width 0.25) (layer "F.Cu") (net 60))
-  (segment (start 136.135386 53.34) (end 144.78 53.34) (width 0.25) (layer "F.Cu") (net 60))
+  (segment (start 144.526 52.959) (end 142.3924 52.959) (width 0.25) (layer "F.Cu") (net 60))
+  (segment (start 146.05 51.435) (end 144.526 52.959) (width 0.25) (layer "F.Cu") (net 60))
   (segment (start 146.05 51.435) (end 148.59 51.435) (width 0.25) (layer "F.Cu") (net 60))
-  (segment (start 144.78 53.34) (end 146.05 52.07) (width 0.25) (layer "F.Cu") (net 60))
+  (segment (start 136.135386 53.34) (end 142.0114 53.34) (width 0.25) (layer "F.Cu") (net 60))
+  (segment (start 142.3924 52.959) (end 142.0114 53.34) (width 0.25) (layer "F.Cu") (net 60))
   (segment (start 134.230386 55.245) (end 136.135386 53.34) (width 0.25) (layer "F.Cu") (net 60))
   (via (at 121.285 55.245) (size 0.8) (drill 0.4) (layers "F.Cu" "B.Cu") (net 60))
-  (segment (start 148.27752 78.81848) (end 148.27752 63.44152) (width 0.25) (layer "B.Cu") (net 60))
   (segment (start 121.285 44.45) (end 121.285 55.245) (width 0.25) (layer "B.Cu") (net 60))
-  (segment (start 142.875718 52.705) (end 147.955 52.705) (width 0.25) (layer "B.Cu") (net 60))
+  (segment (start 142.748 59.944) (end 140.97 58.166) (width 0.25) (layer "B.Cu") (net 60))
+  (segment (start 140.97 58.166) (end 140.97 54.1782) (width 0.25) (layer "B.Cu") (net 60))
   (segment (start 118.11 41.275) (end 121.285 44.45) (width 0.25) (layer "B.Cu") (net 60))
   (segment (start 144.78 59.944) (end 142.748 59.944) (width 0.25) (layer "B.Cu") (net 60))
-  (segment (start 140.97 58.166) (end 140.97 54.610718) (width 0.25) (layer "B.Cu") (net 60))
   (segment (start 148.27752 63.44152) (end 144.78 59.944) (width 0.25) (layer "B.Cu") (net 60))
-  (segment (start 140.97 54.610718) (end 142.875718 52.705) (width 0.25) (layer "B.Cu") (net 60))
+  (segment (start 142.4432 52.705) (end 147.955 52.705) (width 0.25) (layer "B.Cu") (net 60))
+  (segment (start 140.97 54.1782) (end 142.4432 52.705) (width 0.25) (layer "B.Cu") (net 60))
   (segment (start 147.955 52.705) (end 148.59 52.07) (width 0.25) (layer "B.Cu") (net 60))
-  (segment (start 142.748 59.944) (end 140.97 58.166) (width 0.25) (layer "B.Cu") (net 60))
+  (segment (start 148.27752 78.81848) (end 148.27752 63.44152) (width 0.25) (layer "B.Cu") (net 60))
   (segment (start 148.59 52.07) (end 148.59 51.435) (width 0.25) (layer "B.Cu") (net 60))
   (segment (start 146.246 80.85) (end 148.27752 78.81848) (width 0.25) (layer "B.Cu") (net 60))
