File: Northstar 8088 card/ADV-16 CPU/ADV-16 CPU.kicad_sch (KiCad schematic)
At the start: 34 parts, among them J1 Power In, P1 northstar card edge, U11 74LS373, U12 8088-2, U13 74LS00, U14 74LS04, U16 74LS08, U17 8284, U21 74LS153, U22 74LS74, U27 6309-1, U28 74LS373, U29 74LS245, U30 74LS244, U31 74LS10, U4 74LS04, U42 74LS374, U43 74LS373, U44 74LS138, U5 74LS32, U8 74LS74, Y1 24MHz

Commit message: started layout
Parts:
- removed J1: Power In, symbol Connector:Conn_01x03_Pin
- removed P1: northstar card edge, Evan's misc parts:northstar edge connector, symbol Connector_Generic:Conn_02x15_Odd_Even
- removed R1, R2: 510, symbol Device:R
- removed R10: 1K, symbol Device:R
- removed R12: 4.7K, symbol Device:R
- removed TP1: +5V, symbol Connector:Conn_01x01_Pin
- removed TP2: GND, symbol Connector:Conn_01x01_Pin
- removed TP3: CLK, symbol Connector:Conn_01x01_Pin
- removed TP4: RST, symbol Connector:Conn_01x01_Pin
- removed TP5: RDY, symbol Connector:Conn_01x01_Pin
- removed TP6: IFLG, symbol Connector:Conn_01x01_Pin
- removed TP7: OFLG, symbol Connector:Conn_01x01_Pin
- removed U11, U28, U43: 74LS373, symbol 74xx:74LS373
- removed U12: 8088-2, Package_DIP:DIP-40_W15.24mm, symbol MCU_Intel:8088
- removed U13: 74LS00, symbol 74xx:74LS00
- removed U14, U4: 74LS04, symbol 74xx:74LS04
- removed U16: 74LS08, symbol 74xx:74LS08
- removed U17: 8284, Package_DIP:DIP-18_W7.62mm, symbol Timer:8284
- removed U21: 74LS153, symbol 74xx:74LS153
- removed U22, U8: 74LS74, symbol 74xx:74LS74
- removed U27: 6309-1, Package_DIP:DIP-20_W7.62mm, symbol Evan's parts:82S135
- removed U29: 74LS245, symbol 74xx:74LS245
- removed U30: 74LS244, symbol 74xx:74LS244_Split
- removed U31: 74LS10, symbol 74xx:74LS10
- removed U42: 74LS374, symbol 74xx:74LS374
- removed U44: 74LS138, symbol 74xx:74LS138
- removed U5: 74LS32, symbol 74xx:74LS32
- removed W1: +5v EXT, symbol Connector:Conn_01x03_Pin
- removed Y1: 24MHz, symbol Device:Crystal
Connections:
- no-connect marks 21 -> 0
Other:
- added sheet page 1 (ADV-16 CPU pg1.kicad_sch)
- added sheet page 2 (ADV-16 CPU pg2.kicad_sch)
