File: Northstar 8088 card/ADV-16 CPU/ADV-16 CPU pg2.kicad_sch (KiCad schematic)
At the start: 83 parts, among them J2 Conn_01x16_Socket, J3 Conn_01x18_Socket, Q1 2N3904, U1 4164, U1 74LS175, U10 74LS155, U13 74LS00, U14 74LS04, U15 74LS393, U16 74S08, U18 74LS258, U19 74LS174, U2 4164, U2 74S112, U20 74LS03, U22 74LS74, U23 74S00, U24 74LS393, U25 74LS244, U26 74LS258, U3 4164, U3 85ns_Delay, U30 74LS244, U31 74LS10, U4 4164, U4 74S04, U41 74LS280, U5 4164, U6 4164, U6 74LS74, U7 4164, U7 74LS20, U8 4164, U9 4164, U9 74LS00

Commit message: more routing
Connections:
- net GND: now also C2.2, J2.2 (Pin_2), J2.3 (Pin_3), J2.4 (Pin_4)
Changed lines of the file:
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@@
   (junction (at 62.23 76.2) (diameter 0) (color 0 0 0 0)
   )
+  (junction (at 290.195 39.37) (diameter 0) (color 0 0 0 0)
+  )
   (junction (at 391.16 209.55) (diameter 0) (color 0 0 0 0)
   )
@@
         )
       )
+    )
+  )
+  (symbol (lib_id "power:GND") (at 290.195 39.37 0) (unit 1)
+    (in_bom yes) (on_board yes) (dnp no) (fields_autoplaced)
+    (property "Reference" "#PWR023" (at 290.195 45.72 0)
+      (effects (font (size 1.27 1.27)) hide)
+    )
+    (property "Value" "GND" (at 290.195 43.5055 0)
+      (effects (font (size 1.27 1.27)))
+    )
+    (property "Footprint" "" (at 290.195 39.37 0)
+      (effects (font (size 1.27 1.27)) hide)
+    )
+    (property "Datasheet" "" (at 290.195 39.37 0)
+      (effects (font (size 1.27 1.27)) hide)
+    )
+    (pin "1")
+    (instances
+      (project "ADV-16 CPU"
+        (path "/a752c0c4-4fb2-47b8-9f01-e1cc48260014"
+          (reference "#PWR023") (unit 1)
+        )
+        (path "/a752c0c4-4fb2-47b8-9f01-e1cc48260014/c4fe2f20-36ef-4e71-9ba3-72e4f97783f2"
+          (reference "#PWR017") (unit 1)
+        )
+      )
