File: 8087 adapter PCB/8087 adapter PCB.kicad_pcb (KiCad board)
At the start: 2 copper layers, 53.3 x 51.4 mm, 10 parts, among them J3 E2, J4 E1, P2-1 MINT, P2-2 RQ/GT1A, U1 8087, U2 8086/8088

Commit message: tweaks for production
Other:
- outline, holes or cut-outs redrawn
- board text added: "Replica from 2023"
- board text removed: "MADE IN U.S.A."
