File: Northstar HD-5/Northstar HD-5.kicad_sch (KiCad schematic)
At the start: 20 parts, among them P1 Conn_02x15_Odd_Even, U4K 74LS244, U4L 74LS244, U4M 74LS244, U5L 74LS138, U5M 74LS138

Commit message: added some hard drive stuff and tweaked PIO silk
Parts:
- added C12, C13: 0.1uF, symbol Device:C
- added C3: 330pF, symbol Device:C
- added C4: 33pF, symbol Device:C
- added C9: 22uF, symbol Device:C_Polarized
- added CR3: 1N4148, Diode_THT:D_DO-35_SOD27_P7.62mm_Horizontal, symbol Diode:1N4148
- added Q1: 2N3904, Package_TO_SOT_THT:TO-92_Inline, symbol Transistor_BJT:2N3904
- added R23: 3.3K, symbol Device:R
- added R24: 61.9K, symbol Device:R
- added R25: 57.6K, symbol Device:R
- added R26: 5.6K, symbol Device:R
- added R27: 2.2K, symbol Device:R
- added R5, R6: 470R, symbol Device:R
- added RN2: 4.7K, Resistor_THT:R_Array_SIP9, symbol Device:R_Network08
- added TP2: 10Mhz, Connector_Pin:Pin_D1.0mm_L10.0mm, symbol Connector_Generic:Conn_01x01
- added U1C: 74S10, symbol 74xx:74LS10
- added U1D: 74S00, symbol 74xx:74LS00
- added U1F: 74S04, symbol 74xx:74LS04
- added U1K: LM393, symbol Comparator:LM393
- added U1L: 7438, symbol 74xx:74LS38
- added U2D: 74LS175, symbol 74xx:74LS175
- added U2E: 82S129, symbol Evan's misc parts:82S129
- added U2F: 74S174, symbol 74xx:74LS174
- added U2J, U2K: 74LS393, symbol 74xx:74LS393
- added U2L, U2M: 2114, symbol cbm:2114
- added U3K: 74LS164, DIP794W53P254L1930H508Q14N, symbol mouser:SN74LS164N
- added U3L, U?: 74LS374, symbol 74xx:74LS374
- added U3M: 74LS166, symbol 74xx:74LS166
- added U4J: 74LS04, symbol 74xx:74LS04
- added XTL1: 10MHZ, symbol Device:Crystal
Connections:
- net +12V: now also C13.1, CR3.1 (K), R23.1, U1K.8 (V+)
- net +5V: now also C12.1, R27.1, RN2.1 (common), U1C.14 (VCC), U1D.14 (VCC), U1F.14 (VCC), U1K.2 (-), U1L.14 (VCC), U2D.16 (VCC), U2E.16 (Vcc), U2F.16 (VCC), U2J.14 (VCC), U2K.14 (VCC), U2L.18 (Vcc), U2M.18 (Vcc), U3K.14 (VCC), U3L.20 (VCC), U3M.16 (VCC), U4J.14 (VCC), U?.20 (VCC)
- net GND: now also C12.2, C13.2, C4.2, C9.2, Q1.1 (E), R25.2, U1C.7 (GND), U1D.7 (GND), U1F.7 (GND), U1K.4 (V-), U1L.7 (GND), U2D.8 (GND), U2E.13 (/CE1), U2E.14 (/CE2), U2E.15 (A7), U2E.8 (Gnd), U2F.8 (GND), U2J.7 (GND), U2K.7 (GND), U2L.9 (Gnd), U2M.9 (Gnd), U3K.7 (GND), U3L.10 (GND), U3M.1 (Ds), U3M.6 (CE), U3M.8 (GND), U4J.7 (GND), U?.1 (OE), U?.10 (GND)
- net ID 0: now also U2L.14 (D0)
- net ID 1: now also U2L.13 (D1)
- net ID 2: now also U2L.12 (D2)
- net ID 3: now also U2L.11 (D3)
- net ID 4: now also U2M.14 (D0)
- net ID 5: now also U2M.13 (D1)
- net ID 6: now also U2M.12 (D2)
- net ID 7: now also U2M.11 (D3)
- net /CLR ADD: now also U4J.3
- net /LD CONT: now also U?.11 (Cp)
- net ID4: now reaches U4L.12 (O3a)
- net ID4: now also RN2.3 (R2), U3L.9 (O3), U3M.10 (E), U?.3 (D0)
- net ID5: now reaches U4L.14 (O2a)
- net ID5: now also RN2.4 (R3), U3L.6 (O2), U3M.11 (F), U?.4 (D1)
- net ID6: now reaches U4L.16 (O1a)
- net ID6: now also RN2.7 (R6), U3L.5 (O1), U3M.12 (G), U?.7 (D2)
- net ID7: now reaches U4L.18 (O0a)
- net ID7: now also RN2.8 (R7), U3L.2 (O0), U3M.14 (H), U?.8 (D3)
- net ID0: now reaches U4L.3 (O3b)
- net ID0: now also RN2.2 (R1), U3L.19 (O7), U3M.2 (A), U?.18 (D7)
- net ID1: now reaches U4L.5 (O2b)
- net ID1: now also RN2.5 (R4), U3L.16 (O6), U3M.3 (B), U?.17 (D6)
- net ID2: now reaches U4L.7 (O1b)
- net ID2: now also RN2.6 (R5), U3L.15 (O5), U3M.4 (C), U?.14 (D5)
- net ID3: now reaches U4L.9 (O0b)
- net ID3: now also RN2.9 (R8), U3L.12 (O4), U3M.5 (D), U?.13 (D4)
- new net: U1C.4, U1D.11
- new net: U1D.12, U2D.10 (Q2)
- new net: U1C.5, U1D.8
- new net: U1D.9, U2D.15 (Q3)
- new net: U1L.10, U1L.9, U?.15 (O5)
- new net: U1L.1, U1L.2, U?.2 (O0)
- new net: U1L.4, U1L.5, U?.6 (O2)
- new net: C9.1, CR3.2 (A), R23.2, R24.1
- new net: U2J.2 (MR), U2K.12 (MR), U2K.2 (MR), U4J.4
- new net: U2K.13 (CP), U4J.10
- new net: R24.2, R25.1, U1K.3 (+)
- new net: R5.2, U1F.2, XTL1.1
- new net: C4.1, R6.1, U1F.13, XTL1.2
- new net: TP2.1 (Pin_1), U1F.4, U2D.9 (Cp)
- new net: C3.2, R6.2, U1F.12, U1F.3
- new net: C3.1, R5.1, U1F.1
- new net: U1C.3, U1D.3
- new net: Q1.2 (B), R26.1, U1K.1
- new net: U2D.5 (D1), U2E.10 (Q3)
- new net: U2D.12 (D2), U2E.11 (Q2)
- new net: U2D.13 (D3), U2E.12 (Q1)
- new net: U2E.4 (A3), U2F.12 (Q4)
- new net: U2E.5 (A0), U2F.5 (Q1), U2F.6 (D2)
- new net: U2E.6 (A1), U2F.11 (D3), U2F.7 (Q2)
- new net: U2E.7 (A2), U2F.10 (Q3), U2F.13 (D4)
- new net: U1D.1, U2D.7 (Q1)
- new net: U2F.14 (D5), U2F.2 (Q0)
- new net: U2D.3 (~{Q0}), U2D.4 (D0)
- new net 1WR GATE: R26.2, R27.2, U2E.2 (A5), U3M.9 (Clr)
- new net 5MHz: U2D.2 (Q0), U2E.3 (A4), U2F.9 (Cp), U3M.7 (Clk)
- new net HEADER READ: U?.9 (O3)
- new net HS0: U?.19 (O7)
- new net HS1: U?.16 (O6)
- new net PU 3: U2D.1 (~{Mr}), U2F.1 (~{Mr})
- new net RA0: U2K.11 (Q0), U2L.1 (A6), U2M.1 (A6)
- new net RA1: U2K.10 (Q1), U2L.2 (A5), U2M.2 (A5)
- new net RA2: U2K.9 (Q2), U2L.4 (A3), U2M.4 (A3)
- new net RA3: U2K.1 (CP), U2K.8 (Q3), U2L.6 (A1), U2M.6 (A1)
- new net RA4: U2K.3 (Q0), U2L.17 (A7), U2M.17 (A7)
- new net RA5: U2K.4 (Q1), U2L.3 (A4), U2M.3 (A4)
- new net RA6: U2K.5 (Q2), U2L.5 (A0), U2M.5 (A0)
- new net RA7: U2J.1 (CP), U2K.6 (Q3), U2L.7 (A2), U2M.7 (A2)
- new net RA8: U2J.3 (Q0), U2L.16 (A8), U2M.16 (A8)
- new net RA9: U2J.4 (Q1), U2L.15 (A9), U2M.15 (A9)
- new net RAW INDEX: U2F.3 (D0)
- new net RD CLK: U3K.8 (CLK)
- new net RD GATE: U3K.9 (~{CLR})
- new net SD00: U3K.3 (QA), U3L.18 (D7)
- new net SD01: U3K.4 (QB), U3L.17 (D6)
- new net SD02: U3K.5 (QC), U3L.14 (D5)
- new net SD03: U3K.6 (QD), U3L.13 (D4)
- new net SD04: U3K.10 (QE), U3L.8 (D3)
- new net SD05: U3K.11 (QF), U3L.7 (D2)
- new net SD06: U3K.12 (QG), U3L.4 (D1)
- new net SD07: U3K.13 (QH), U3L.3 (D0)
- new net SEP RD DATA: U3K.1 (A), U3K.2 (B)
- new net SYNC INDEX: U2F.15 (Q5)
- new net WR DATA: U2F.4 (D1), U3M.13 (Qh)
- new net /DIR / PRCMP: U2E.1 (A6), U?.5 (O1)
- new net /HS2: U1L.8
- new net /LD WR BYTE: U3M.15 (PE)
- new net /LOW CUR: U?.12 (O4)
- new net /RD BYT RDY: U3L.11 (Cp)
- new net /RD DATA TO RAM: U3L.1 (OE)
- new net /SEL RAM: U2L.8 (~{CS}), U2M.8 (~{CS}), U4J.11
- new net /STEP: U1L.3
- new net /WR GATE: Q1.3 (C)
- new net /WR RAM: U2L.10 (R/~{W}), U2M.10 (R/~{W})
- no-connect marks 8 -> 15
Other:
- note added: "Double check here on schematic vs real board"
- note added: "Drive Control Latch"
- note added: "Parallel to serial converter"
- note added: "RAM address counter"
- note added: "Read Data Buffer"
- note added: "Serial to parallel converter"
- note added: "These address and data lines can be juggled for layout purposes"
- note added: "these can be mixed as long as inputs match outputs"
- moved on the sheet: RN1

Commit message: hd5 stuff and pio gerbers
Parts:
- removed C1: 22uF, Capacitor_THT:CP_Radial_D5.0mm_P2.50mm, symbol Device:C_Polarized
- removed C12, C13: 0.1uF, symbol Device:C
- removed C2, C7: 6.8uF, Capacitor_THT:CP_Radial_D5.0mm_P2.50mm, symbol Device:C_Polarized
- removed C3: 330pF, symbol Device:C
- removed C4: 33pF, symbol Device:C
- removed C9: 22uF, symbol Device:C_Polarized
- removed C? (x2): *, Capacitor_THT:C_Disc_D7.5mm_W2.5mm_P5.00mm, symbol Device:C
- removed CR3: 1N4148, Diode_THT:D_DO-35_SOD27_P7.62mm_Horizontal, symbol Diode:1N4148
- removed P1: Conn_02x15_Odd_Even, Evan's misc parts:northstar edge connector, symbol Connector_Generic:Conn_02x15_Odd_Even
- removed Q1: 2N3904, Package_TO_SOT_THT:TO-92_Inline, symbol Transistor_BJT:2N3904
- removed R1, R2, R3, R4: 1k, Resistor_THT:R_Axial_DIN0207_L6.3mm_D2.5mm_P15.24mm_Horizontal, symbol Device:R
- removed R23: 3.3K, symbol Device:R
- removed R24: 61.9K, symbol Device:R
- removed R25: 57.6K, symbol Device:R
- removed R26: 5.6K, symbol Device:R
- removed R27: 2.2K, symbol Device:R
- removed R5, R6: 470R, symbol Device:R
- removed RN1: 220/330, Resistor_THT:R_Array_SIP8, symbol Device:R_Network_Dividers_x06_SIP
- removed RN2: 4.7K, Resistor_THT:R_Array_SIP9, symbol Device:R_Network08
- removed TP2: 10Mhz, Connector_Pin:Pin_D1.0mm_L10.0mm, symbol Connector_Generic:Conn_01x01
- removed TP5: 5v PLL, Connector_Pin:Pin_D1.0mm_L10.0mm, symbol Connector_Generic:Conn_01x01
- removed TP7: 5v, Connector_Pin:Pin_D1.0mm_L10.0mm, symbol Connector_Generic:Conn_01x01
- removed TP8: Gnd, Connector_Pin:Pin_D1.0mm_L10.0mm, symbol Connector_Generic:Conn_01x01
- removed U1C: 74S10, symbol 74xx:74LS10
- removed U1D: 74S00, symbol 74xx:74LS00
- removed U1F: 74S04, symbol 74xx:74LS04
- removed U1K: LM393, symbol Comparator:LM393
- removed U1L: 7438, symbol 74xx:74LS38
- removed U2D: 74LS175, symbol 74xx:74LS175
- removed U2E: 82S129, symbol Evan's misc parts:82S129
- removed U2F: 74S174, symbol 74xx:74LS174
- removed U2J, U2K: 74LS393, symbol 74xx:74LS393
- removed U2L, U2M: 2114, symbol cbm:2114
- removed U3K: 74LS164, DIP794W53P254L1930H508Q14N, symbol mouser:SN74LS164N
- removed U3L, U?: 74LS374, symbol 74xx:74LS374
- removed U3M: 74LS166, symbol 74xx:74LS166
- removed U4J: 74LS04, symbol 74xx:74LS04
- removed U4K, U4L, U4M: 74LS244, symbol 74xx:74LS244
- removed U5L, U5M: 74LS138, symbol 74xx:74LS138
- removed VR1: LM340AT-5, Package_TO_SOT_THT:TO-220-3_Vertical, symbol Regulator_Linear:LM341T-05_TO220
- removed XTL1: 10MHZ, symbol Device:Crystal
Connections:
- no-connect marks 15 -> 0
Other:
- added sheet HD5 Sheet 1 (hd5 sheet1.kicad_sch)
- added sheet HD5 Sheet 2 (hd5 sheet2.kicad_sch)
- added sheet HD5 Spare Gates (hd5 spare.kicad_sch)
- added sheet Power and pullups (hd5 power.kicad_sch)
- note removed: "Double check here on schematic vs real board"
- note removed: "Drive Control Latch"
- note removed: "Host Data Drivers"
- note removed: "Host Data Receiver"
- note removed: "I/O Address Decoders"
- note removed: "Parallel to serial converter"
- note removed: "RAM address counter"
- note removed: "Read Data Buffer"
- note removed: "Serial to parallel converter"
- note removed: "Status Register"
- note removed: "These address and data lines can be juggled for layout purposes"
- note removed: "these can be mixed as long as inputs match outputs"
