File: Northstar HD-5/hd5 spare.kicad_sch (KiCad schematic)
At the start: 9 parts, among them U1C 74S10, U1F 74S04, U1K LM393, U1L 7438, U3D 74LS04, U4D 74S04, U4J 74LS04, U5H 74LS32, U5J 74LS00

Commit message: changes to hd-5 and gitignore
Parts:
- U1C1: renamed from U1C; footprint (none) -> Package_DIP:DIP-14_W7.62mm
- U1F1: renamed from U1F; footprint (none) -> Package_DIP:DIP-14_W7.62mm
- U1K1: renamed from U1K; footprint (none) -> Package_DIP:DIP-8-16_W7.62mm
- U1L1: renamed from U1L; footprint (none) -> Package_DIP:DIP-14_W7.62mm
- U3D1: renamed from U3D; footprint (none) -> Package_DIP:DIP-14_W7.62mm
- U4D1: renamed from U4D; footprint (none) -> Package_DIP:DIP-14_W7.62mm
- U4J1: renamed from U4J; footprint (none) -> Package_DIP:DIP-14_W7.62mm
- U5H1: renamed from U5H; footprint (none) -> Package_DIP:DIP-14_W7.62mm
- U5J1: renamed from U5J; footprint (none) -> Package_DIP:DIP-14_W7.62mm
Changed lines of the file:
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@@
   (symbol (lib_id "74xx:74LS04") (at 146.685 66.675 0) (unit 4)
     (in_bom yes) (on_board yes) (fields_autoplaced)
-    (property "Reference" "U4J" (id 0) (at 146.685 58.8985 0))
+    (property "Reference" "U4J1" (id 0) (at 146.685 58.8985 0))
     (property "Value" "74LS04" (id 1) (at 146.685 61.6736 0))
-    (property "Footprint" "" (id 2) (at 146.685 66.675 0)
+    (property "Footprint" "Package_DIP:DIP-14_W7.62mm" (id 2) (at 146.685 66.675 0)
       (effects (font (size 1.27 1.27)) hide)
     )
@@
   (symbol (lib_id "Comparator:LM393") (at 166.37 97.155 0) (unit 2)
     (in_bom yes) (on_board yes) (fields_autoplaced)
-    (property "Reference" "U1K" (id 0) (at 166.37 88.1085 0))
+    (property "Reference" "U1K1" (id 0) (at 166.37 88.1085 0))
     (property "Value" "LM393" (id 1) (at 166.37 90.8836 0))
-    (property "Footprint" "" (id 2) (at 166.37 97.155 0)
+    (property "Footprint" "Package_DIP:DIP-8-16_W7.62mm" (id 2) (at 166.37 97.155 0)
       (effects (font (size 1.27 1.27)) hide)
     )
@@
   (symbol (lib_id "74xx:74LS04") (at 127.635 90.805 0) (unit 5)
     (in_bom yes) (on_board yes) (fields_autoplaced)
-    (property "Reference" "U4D" (id 0) (at 127.635 83.0285 0))
+    (property "Reference" "U4D1" (id 0) (at 127.635 83.0285 0))
     (property "Value" "74S04" (id 1) (at 127.635 85.8036 0))
-    (property "Footprint" "" (id 2) (at 127.635 90.805 0)
+    (property "Footprint" "Package_DIP:DIP-14_W7.62mm" (id 2) (at 127.635 90.805 0)
       (effects (font (size 1.27 1.27)) hide)
     )
@@
   (symbol (lib_id "74xx:74LS38") (at 166.37 69.215 0) (unit 4)
     (in_bom yes) (on_board yes) (fields_autoplaced)
-    (property "Reference" "U1L" (id 0) (at 166.37 61.4385 0))
+    (property "Reference" "U1L1" (id 0) (at 166.37 61.4385 0))
     (property "Value" "7438" (id 1) (at 166.37 64.2136 0))
-    (property "Footprint" "" (id 2) (at 166.37 69.215 0)
+    (property "Footprint" "Package_DIP:DIP-14_W7.62mm" (id 2) (at 166.37 69.215 0)
       (effects (font (size 1.27 1.27)) hide)
     )
@@
   (symbol (lib_id "74xx:74LS00") (at 185.42 82.55 0) (unit 3)
     (in_bom yes) (on_board yes) (fields_autoplaced)
-    (property "Reference" "U5J" (id 0) (at 185.42 74.7735 0))
+    (property "Reference" "U5J1" (id 0) (at 185.42 74.7735 0))
     (property "Value" "74LS00" (id 1) (at 185.42 77.5486 0))
-    (property "Footprint" "" (id 2) (at 185.42 82.55 0)
+    (property "Footprint" "Package_DIP:DIP-14_W7.62mm" (id 2) (at 185.42 82.55 0)
       (effects (font (size 1.27 1.27)) hide)
     )
@@
   (symbol (lib_id "74xx:74LS04") (at 127.635 102.87 0) (unit 6)
     (in_bom yes) (on_board yes) (fields_autoplaced)
-    (property "Reference" "U4D" (id 0) (at 127.635 95.0935 0))
+    (property "Reference" "U4D1" (id 0) (at 127.635 95.0935 0))
     (property "Value" "74S04" (id 1) (at 127.635 97.8686 0))
-    (property "Footprint" "" (id 2) (at 127.635 102.87 0)
+    (property "Footprint" "Package_DIP:DIP-14_W7.62mm" (id 2) (at 127.635 102.87 0)
       (effects (font (size 1.27 1.27)) hide)
     )
@@
   (symbol (lib_id "74xx:74LS04") (at 127.635 78.74 0) (unit 4)
     (in_bom yes) (on_board yes) (fields_autoplaced)
-    (property "Reference" "U4D" (id 0) (at 127.635 70.9635 0))
+    (property "Reference" "U4D1" (id 0) (at 127.635 70.9635 0))
     (property "Value" "74S04" (id 1) (at 127.635 73.7386 0))
-    (property "Footprint" "" (id 2) (at 127.635 78.74 0)
+    (property "Footprint" "Package_DIP:DIP-14_W7.62mm" (id 2) (at 127.635 78.74 0)
       (effects (font (size 1.27 1.27)) hide)
     )
@@
   (symbol (lib_id "74xx:74LS04") (at 127.635 66.675 0) (unit 3)
     (in_bom yes) (on_board yes) (fields_autoplaced)
-    (property "Reference" "U4D" (id 0) (at 127.635 58.8985 0))
+    (property "Reference" "U4D1" (id 0) (at 127.635 58.8985 0))
     (property "Value" "74S04" (id 1) (at 127.635 61.6736 0))
-    (property "Footprint" "" (id 2) (at 127.635 66.675 0)
+    (property "Footprint" "Package_DIP:DIP-14_W7.62mm" (id 2) (at 127.635 66.675 0)
       (effects (font (size 1.27 1.27)) hide)
     )
@@
   (symbol (lib_id "74xx:74LS04") (at 108.585 79.375 0) (unit 2)
     (in_bom yes) (on_board yes) (fields_autoplaced)
-    (property "Reference" "U3D" (id 0) (at 108.585 71.5985 0))
+    (property "Reference" "U3D1" (id 0) (at 108.585 71.5985 0))
     (property "Value" "74LS04" (id 1) (at 108.585 74.3736 0))
-    (property "Footprint" "" (id 2) (at 108.585 79.375 0)
+    (property "Footprint" "Package_DIP:DIP-14_W7.62mm" (id 2) (at 108.585 79.375 0)
       (effects (font (size 1.27 1.27)) hide)
     )
@@
   (symbol (lib_id "74xx:74LS04") (at 147.32 90.805 0) (unit 5)
     (in_bom yes) (on_board yes) (fields_autoplaced)
-    (property "Reference" "U1F" (id 0) (at 147.32 83.0285 0))
+    (property "Reference" "U1F1" (id 0) (at 147.32 83.0285 0))
     (property "Value" "74S04" (id 1) (at 147.32 85.8036 0))
-    (property "Footprint" "" (id 2) (at 147.32 90.805 0)
+    (property "Footprint" "Package_DIP:DIP-14_W7.62mm" (id 2) (at 147.32 90.805 0)
       (effects (font (size 1.27 1.27)) hide)
     )
@@
   (symbol (lib_id "74xx:74LS10") (at 166.37 82.55 0) (unit 1)
     (in_bom yes) (on_board yes) (fields_autoplaced)
-    (property "Reference" "U1C" (id 0) (at 166.37 74.7735 0))
+    (property "Reference" "U1C1" (id 0) (at 166.37 74.7735 0))
     (property "Value" "74S10" (id 1) (at 166.37 77.5486 0))
-    (property "Footprint" "" (id 2) (at 166.37 82.55 0)
+    (property "Footprint" "Package_DIP:DIP-14_W7.62mm" (id 2) (at 166.37 82.55 0)
       (effects (font (size 1.27 1.27)) hide)
     )
@@
   (symbol (lib_id "74xx:74LS32") (at 185.42 69.215 0) (unit 1)
     (in_bom yes) (on_board yes) (fields_autoplaced)
-    (property "Reference" "U5H" (id 0) (at 185.42 61.4385 0))
+    (property "Reference" "U5H1" (id 0) (at 185.42 61.4385 0))
     (property "Value" "74LS32" (id 1) (at 185.42 64.2136 0))
-    (property "Footprint" "" (id 2) (at 185.42 69.215 0)
+    (property "Footprint" "Package_DIP:DIP-14_W7.62mm" (id 2) (at 185.42 69.215 0)
       (effects (font (size 1.27 1.27)) hide)
     )
@@
   (symbol (lib_id "74xx:74LS04") (at 108.585 66.675 0) (unit 1)
     (in_bom yes) (on_board yes) (fields_autoplaced)
-    (property "Reference" "U3D" (id 0) (at 108.585 58.8985 0))
+    (property "Reference" "U3D1" (id 0) (at 108.585 58.8985 0))
     (property "Value" "74LS04" (id 1) (at 108.585 61.6736 0))
-    (property "Footprint" "" (id 2) (at 108.585 66.675 0)
+    (property "Footprint" "Package_DIP:DIP-14_W7.62mm" (id 2) (at 108.585 66.675 0)
       (effects (font (size 1.27 1.27)) hide)
     )
@@
   (symbol (lib_id "74xx:74LS04") (at 146.685 78.74 0) (unit 3)
     (in_bom yes) (on_board yes) (fields_autoplaced)
-    (property "Reference" "U1F" (id 0) (at 146.685 70.9635 0))
+    (property "Reference" "U1F1" (id 0) (at 146.685 70.9635 0))
     (property "Value" "74S04" (id 1) (at 146.685 73.7386 0))
-    (property "Footprint" "" (id 2) (at 146.685 78.74 0)
+    (property "Footprint" "Package_DIP:DIP-14_W7.62mm" (id 2) (at 146.685 78.74 0)
       (effects (font (size 1.27 1.27)) hide)
     )
@@
   (symbol (lib_id "74xx:74LS04") (at 108.585 91.44 0) (unit 6)
     (in_bom yes) (on_board yes) (fields_autoplaced)
-    (property "Reference" "U3D" (id 0) (at 108.585 83.6635 0))
+    (property "Reference" "U3D1" (id 0) (at 108.585 83.6635 0))
     (property "Value" "74LS04" (id 1) (at 108.585 86.4386 0))
-    (property "Footprint" "" (id 2) (at 108.585 91.44 0)
+    (property "Footprint" "Package_DIP:DIP-14_W7.62mm" (id 2) (at 108.585 91.44 0)
       (effects (font (size 1.27 1.27)) hide)
     )

Commit message: placed components and repaired multi sheet labels
Parts:
- U1K1: footprint Package_DIP:DIP-8-16_W7.62mm -> Package_DIP:DIP-8_W7.62mm
Changed lines of the file:
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@@
     (property "Reference" "U1K1" (id 0) (at 166.37 88.1085 0))
     (property "Value" "LM393" (id 1) (at 166.37 90.8836 0))
-    (property "Footprint" "Package_DIP:DIP-8-16_W7.62mm" (id 2) (at 166.37 97.155 0)
+    (property "Footprint" "Package_DIP:DIP-8_W7.62mm" (id 2) (at 166.37 97.155 0)
       (effects (font (size 1.27 1.27)) hide)
     )
