File: Northstar SIO/Northstar SIO.kicad_sch (KiCad schematic)
At the start: 50 parts, among them J1 DB25_Female, J1A Clock Header, J3A Configuration Header, U1B 74LS161, U1C 74LS161, U1D 74LS161, U1E 74LS174, U2A MC1489PG, U2B 74LS04, U2C 74LS109, U2D 74LS175, U2E 74LS243, U3B 74LS00, U3C 74LS138, U3D 74LS03, U3E 74LS243, U4A MC1488N, U4E 8251A

Commit message: laid out SIO board
Parts:
- removed C? (x3): 0.047uF, symbol Device:C
- added C16, C20, C7: 0.047uF, Capacitor_THT:C_Disc_D7.5mm_W2.5mm_P5.00mm, symbol Device:C
- C1, C2, C3: footprint (none) -> Capacitor_THT:CP_Radial_D5.0mm_P2.50mm
- C10, C11, C12, C13, C14, C15, C17, C18, C19, C8, C9: renamed from C?; footprint (none) -> Capacitor_THT:C_Disc_D7.5mm_W2.5mm_P5.00mm
- C4, C5, C6: footprint (none) -> Capacitor_THT:C_Disc_D7.5mm_W2.5mm_P5.00mm
- J1: footprint (none) -> Evan's misc parts:northstar db25
- J1A1: renamed from J1A; footprint (none) -> Package_DIP:DIP-8_W7.62mm
- J2: renamed from J?; footprint (none) -> Evan's misc parts:northstar edge connector
- J3A1: renamed from J3A; footprint (none) -> Package_DIP:DIP-16_W7.62mm
- R1, R2, R3, R4, R5, R6: footprint (none) -> Resistor_THT:R_Axial_DIN0207_L6.3mm_D2.5mm_P15.24mm_Horizontal
- R10, R7, R8, R9: renamed from R?; footprint (none) -> Resistor_THT:R_Axial_DIN0207_L6.3mm_D2.5mm_P15.24mm_Horizontal
- U1B1: renamed from U1B; footprint (none) -> Package_DIP:DIP-16_W7.62mm
- U1C1: renamed from U1C; footprint (none) -> Package_DIP:DIP-16_W7.62mm
- U1D1: renamed from U1D; footprint (none) -> Package_DIP:DIP-16_W7.62mm
- U1E1: renamed from U1E; footprint (none) -> Package_DIP:DIP-16_W7.62mm
- U2A1: renamed from U2A; footprint DIP254P762X469-14 -> Package_DIP:DIP-14_W7.62mm
- U2B1: renamed from U2B; footprint (none) -> Package_DIP:DIP-14_W7.62mm
- U2C1: renamed from U2C; footprint (none) -> Package_DIP:DIP-16_W7.62mm
- U2D1: renamed from U2D; footprint (none) -> Package_DIP:DIP-16_W7.62mm
- U2E1: renamed from U2E; footprint (none) -> Package_DIP:DIP-12_W7.62mm
- U3B1: renamed from U3B; footprint (none) -> Package_DIP:DIP-14_W7.62mm
- U3C1: renamed from U3C; footprint (none) -> Package_DIP:DIP-16_W7.62mm
- U3D1: renamed from U3D; footprint (none) -> Package_DIP:DIP-14_W7.62mm
- U3E1: renamed from U3E; footprint (none) -> Package_DIP:DIP-12_W7.62mm
- U4A1: renamed from U4A; footprint DIP794W45P254L1969H508Q14 -> Package_DIP:DIP-14_W7.62mm
- U4E1: renamed from U4E; footprint DIL28-6 -> Package_DIP:DIP-28_W15.24mm
- W1: footprint (none) -> Connector_PinHeader_2.54mm:PinHeader_1x03_P2.54mm_Vertical
Connections:
- net +12V: now also C20.1
- net +5V: now also C16.1
- net -12V: now also C7.1
- net B: now also J3A1.4 (Pin_4), W1.2 (Pin_2)
- net GND: now also C16.2, C20.2, C7.2
- net RCD: now reaches C12.2, R10.1, U2A1.12 (RESPONSE_COTROL_D)
- net RCC: now reaches C14.2, R9.1, U2A1.9 (RESPONSE_COTROL_C)
- net RCB: now reaches C13.2, R8.1, U2A1.5 (RESPONSE_COTROL_B)
- net RCA: now reaches C11.2, R7.1, U2A1.2 (RESPONSE_COTROL_A)
- new net: J3A1.7 (Pin_7), R6.2
- new net: J1.2, J3A1.6 (Pin_6)
- new net: J1A1.4 (Pin_4), J3A1.8 (Pin_8), U4E1.25 (~{RXC})
Other:
- moved on the sheet: C1, C2, C3, R1
